File: hardware/kicad/power.kicad_sch (KiCad schematic)
At the start: 26 parts, among them J1 36V IN, Q1 SQD50P06-15L, U1 LM5164DDAR

Commit message: Complete LCSC part numbers in the BOM
Every BOM line now has an LCSC number except the Pico module (A1), which
is marked "user-supplied, hand-solder". Parts were checked against the
JLCPCB parts library for spec, Basic/Extended status and stock.

- build_schematic.py: RES_PARTS / CAP_PARTS value+footprint lookup tables
  used by R() / C(), which now raise if a passive has no entry; props for
  the diodes, LEDs, logic ICs, PTC (Littelfuse 2920L050DR, 60 V), IDC
  header (ZHOURI DC3-2.54-14PAS), JST-XH 7p and the Omron B3S-1000 reset
  button.
- Regenerated the schematic sheets, kicad/bom.csv, fab BOM and the README
  missing-LCSC table. PCB, CPL, gerbers and drills are unchanged.

Co-Authored-By: Claude Sonnet 5.5 <noreply@anthropic.com>
Parts:
- C10: LCSC (none) -> C57112; MPN (none) -> FH 0603B103K500NT
- C2, C3, C4: LCSC (none) -> C86054; MPN (none) -> Murata GRM32ER72A225KA35L
- C5: LCSC (none) -> C1604; MPN (none) -> FH 0603B222K500NT
- C6: LCSC (none) -> C1613; MPN (none) -> Samsung CL10B332KB8NNNC
- C7: LCSC (none) -> C14858; MPN (none) -> Samsung CL10C101JB8NNNC
- C8, C9: LCSC (none) -> C12891; MPN (none) -> Samsung CL31A226KAHNNNE
- D1: LCSC (none) -> C129730; MPN MMSZ5245B -> onsemi MMSZ5245BT1G
- D3: LCSC (none) -> C12624; MPN (none) -> KENTO KT-0603G
- R1: LCSC (none) -> C31850; MPN (none) -> UNI-ROYAL 0603WAF2202T5E
- R2: LCSC (none) -> C2930101; MPN (none) -> FOJAN FRC0603F4122TS
- R3, R7: LCSC (none) -> C25803; MPN (none) -> UNI-ROYAL 0603WAF1003T5E
- R4: LCSC (none) -> C25967; MPN (none) -> UNI-ROYAL 0603WAF3162T5E
- R5: LCSC (none) -> C25811; MPN (none) -> UNI-ROYAL 0603WAF2003T5E
- R6: LCSC (none) -> C23162; MPN (none) -> UNI-ROYAL 0603WAF4701T5E
- R8: LCSC (none) -> C23234; MPN (none) -> UNI-ROYAL 0603WAF7501T5E
