File: hardware/kicad/clutch.kicad_sch (KiCad schematic)
At the start: 24 parts, among them J4 CLUTCH COIL, Q2 AGM60P20R, Q3 2N7002, Q4 SI2308A, U6 TLV9061

Commit message: Add routed controller PCB, clutch CAD and mill notes
- Schematic: panel ribbon (2x7 IDC) + feed-unit header (JST-XH 7) so all
  connectors fit one 100 mm board edge; fix stub-bridging in the generator.
- PCB (hardware/tools/build_pcb.py): 100x100 mm 4-layer board built from the
  netlist - fixed placement for power/connectors, auto-placed passives,
  GND / split +36V/+3V3 inner planes, Freerouting, post-route power pours,
  GND stitching; fix_planes.py drops plane vias for leftovers;
  check_pcb.py runs DRC with schematic parity. 3D renders in hardware/renders.
  Status: 5 unconnected items + 2 starved thermals left for interactive
  routing (see hardware/kicad/drc.json after check_pcb.py).
- mechanical/clutch: parametric build123d model of the DIY tooth clutch
  (field housing, coil, rotor, armature, leaf springs, output hub/shaft,
  cover), STEP/STL export and VTK renders.
- docs/mill.md: SIEG X3.5D research and the measurements still needed.

Co-Authored-By: Claude Opus 5.5 <noreply@anthropic.com>
Parts:
- removed J4: CLUTCH COIL, Connector_Phoenix_MSTB:PhoenixContact_MSTBA_2,5_2-G-5,08_1x02_P5.08mm_Horizontal, symbol Connector:Screw_Terminal_01x02
- added J3: CLUTCH COIL, Connector_Phoenix_MSTB:PhoenixContact_MSTBA_2,5_2-G-5,08_1x02_P5.08mm_Horizontal, symbol Connector:Screw_Terminal_01x02
Connections:
- net COIL_N: now also J3.2 (Pin_2)
- net COIL_P: now also J3.1 (Pin_1)
Changed lines of the file:
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@@
 		(on_board yes)
 		(dnp no)
-		(property "Reference" "J4"
+		(property "Reference" "J3"
 			(at 38.1 96.52 0)
 			(effects
@@
 			(project "power-feed"
 				(path "/8e300617-3fca-5828-bedd-07eaa661f340/fee9f53f-ca95-5009-a118-475b15ee829d"
-					(reference "J4")
+					(reference "J3")
 					(unit 1)
 				)

Commit message: Complete LCSC part numbers in the BOM
Every BOM line now has an LCSC number except the Pico module (A1), which
is marked "user-supplied, hand-solder". Parts were checked against the
JLCPCB parts library for spec, Basic/Extended status and stock.

- build_schematic.py: RES_PARTS / CAP_PARTS value+footprint lookup tables
  used by R() / C(), which now raise if a passive has no entry; props for
  the diodes, LEDs, logic ICs, PTC (Littelfuse 2920L050DR, 60 V), IDC
  header (ZHOURI DC3-2.54-14PAS), JST-XH 7p and the Omron B3S-1000 reset
  button.
- Regenerated the schematic sheets, kicad/bom.csv, fab BOM and the README
  missing-LCSC table. PCB, CPL, gerbers and drills are unchanged.

Co-Authored-By: Claude Sonnet 5.5 <noreply@anthropic.com>
Parts:
- C32: LCSC (none) -> C86054; MPN (none) -> Murata GRM32ER72A225KA35L
- C33: LCSC (none) -> C1588; MPN (none) -> Samsung CL10B102KB8NNNC
- C34: LCSC (none) -> C14663; MPN (none) -> Yageo CC0603KRX7R9BB104
- C35: LCSC (none) -> C57112; MPN (none) -> FH 0603B103K500NT
- D5: LCSC (none) -> C82050; MPN MMSZ5242B -> onsemi MMSZ5242BT1G
- D8: LCSC (none) -> C965802; MPN (none) -> XINGLIGHT XL-1608UYC-06
- F2: LCSC (none) -> C207082; MPN Littelfuse 2920L050/60MR (verify 60 V rating + LCSC) -> Littelfuse 2920L050DR (0.5 A hold, 1 A trip, 60 V)
- R38: LCSC (none) -> C4190; MPN (none) -> UNI-ROYAL 0603WAF2201T5E
- R39: LCSC (none) -> C17936; MPN (none) -> UNI-ROYAL 1206W4F4701T5E
- R40: LCSC (none) -> C22775; MPN (none) -> UNI-ROYAL 0603WAF1000T5E
- R41: LCSC (none) -> C25803; MPN (none) -> UNI-ROYAL 0603WAF1003T5E
- R43: LCSC (none) -> C31850; MPN (none) -> UNI-ROYAL 0603WAF2202T5E
- R44, R47: LCSC (none) -> C21190; MPN (none) -> UNI-ROYAL 0603WAF1001T5E
- R45: LCSC (none) -> C25811; MPN (none) -> UNI-ROYAL 0603WAF2003T5E
- R46: LCSC (none) -> C25804; MPN (none) -> UNI-ROYAL 0603WAF1002T5E

Commit message: Schematic: bare RP2040 instead of the Pico module
RP2040 (QFN-56) per Raspberry Pi's minimal design: W25Q16JV 2 MB QSPI flash, 12 MHz crystal with 1k series,
internal 1.1 V core regulator, BOOTSEL + RESET buttons, JST-SH SWD, status LED on GPIO25, USB-C (5.1k CC,
27R series). +3V3 now from an AP2112K-3.3 fed by VSYS = +5V or USB VBUS through Schottkys. Same GPIO
numbers as the Pico, so the firmware is unchanged. ERC 0 findings, netlist 132 nets / 189 parts match.
Layout follows (PCB agent). LCSC numbers for the flash and crystal still to be verified.

Co-Authored-By: Claude Opus 5.5 <noreply@anthropic.com>
Parts:
- removed C32: 2.2uF 100V, Capacitor_SMD:C_1210_3225Metric, symbol Device:C
- removed C33: 1nF, Capacitor_SMD:C_0603_1608Metric, symbol Device:C
- removed C34: 100nF, Capacitor_SMD:C_0603_1608Metric, symbol Device:C
- removed C35: 10nF, Capacitor_SMD:C_0603_1608Metric, symbol Device:C
- removed D5: 12V, Diode_SMD:D_SOD-123, symbol Device:D_Zener
- removed D6: SS210 (fast decay), Diode_SMD:D_SMA, symbol Device:D_Schottky
- removed J3: CLUTCH COIL, Connector_Phoenix_MSTB:PhoenixContact_MSTBA_2,5_2-G-5,08_1x02_P5.08mm_Horizontal, symbol Connector:Screw_Terminal_01x02
- removed R38: 2.2k, Resistor_SMD:R_0603_1608Metric, symbol Device:R
- removed R39: 4.7k, Resistor_SMD:R_1206_3216Metric, symbol Device:R
- removed R40: 100, Resistor_SMD:R_0603_1608Metric, symbol Device:R
- removed R41: 100k, Resistor_SMD:R_0603_1608Metric, symbol Device:R
- removed R42: 0.1 1% 1W, Resistor_SMD:R_1206_3216Metric, symbol Device:R
- removed R43: 22k, Resistor_SMD:R_0603_1608Metric, symbol Device:R
- removed R44: 1k, Resistor_SMD:R_0603_1608Metric, symbol Device:R
- removed R45: 200k, Resistor_SMD:R_0603_1608Metric, symbol Device:R
- removed R46: 10k, Resistor_SMD:R_0603_1608Metric, symbol Device:R
- removed U6: TLV9061, Package_TO_SOT_SMD:SOT-23-5, symbol Amplifier_Operational:TLV9061xDBV
- added C49: 2.2uF 100V, Capacitor_SMD:C_1210_3225Metric, symbol Device:C
- added C50: 1nF, Capacitor_SMD:C_0603_1608Metric, symbol Device:C
- added C51: 100nF, Capacitor_SMD:C_0603_1608Metric, symbol Device:C
- added C52: 10nF, Capacitor_SMD:C_0603_1608Metric, symbol Device:C
- added D10: yellow, LED_SMD:LED_0603_1608Metric, symbol Device:LED
- added D9: SS210 (freewheel), Diode_SMD:D_SMA, symbol Device:D_Schottky
- added J5: CLUTCH COIL, Connector_Phoenix_MSTB:PhoenixContact_MSTBA_2,5_2-G-5,08_1x02_P5.08mm_Horizontal, symbol Connector:Screw_Terminal_01x02
- added R48: 4.7k, Resistor_SMD:R_1206_3216Metric, symbol Device:R
- added R49: 100, Resistor_SMD:R_0603_1608Metric, symbol Device:R
- added R50: 100k, Resistor_SMD:R_0603_1608Metric, symbol Device:R
- added R51: 0.1 1% 1W, Resistor_SMD:R_1206_3216Metric, symbol Device:R
- added R52: 22k, Resistor_SMD:R_0603_1608Metric, symbol Device:R
- added R53, R56: 1k, Resistor_SMD:R_0603_1608Metric, symbol Device:R
- added R54: 200k, Resistor_SMD:R_0603_1608Metric, symbol Device:R
- added R55: 10k, Resistor_SMD:R_0603_1608Metric, symbol Device:R
- added U9: TLV9061, Package_TO_SOT_SMD:SOT-23-5, symbol Amplifier_Operational:TLV9061xDBV
- D7: value SS210 (freewheel) -> 12V; footprint Diode_SMD:D_SMA -> Diode_SMD:D_SOD-123; symbol Device:D_Schottky -> Device:D_Zener; LCSC C14996 -> C82050; MPN SS210 -> onsemi MMSZ5242BT1G
- D8: value yellow -> SS210 (fast decay); footprint LED_SMD:LED_0603_1608Metric -> Diode_SMD:D_SMA; symbol Device:LED -> Device:D_Schottky; LCSC C965802 -> C14996; MPN XINGLIGHT XL-1608UYC-06 -> SS210
- R47: value 1k -> 2.2k; LCSC C21190 -> C4190; MPN UNI-ROYAL 0603WAF1001T5E -> UNI-ROYAL 0603WAF2201T5E
Connections:
- net +3V3: now also C51.1, U9.5 (V+)
- net CLUTCH_ISENSE: now also C52.1, R56.2; no longer R47.2
- net CLUTCH_LS_GATE: now also R49.1
- net CLUTCH_SHUNT: now also R51.1, R53.1
- net CLUTCH_VIN: now also D7.1 (K), D8.1 (K), R47.2, C49.1
- net COIL_N: now also D8.2 (A), J5.2 (Pin_2)
- net COIL_P: now also D9.1 (K), J5.1 (Pin_1), R52.1; no longer D7.1 (K)
- net GND: now also C49.2, C50.2, C51.2, C52.2, D10.1 (K), D9.2 (A), R50.2, R51.2, R55.2, U9.2 (V-); no longer D7.2 (A), D8.1 (K)
- net HS_GATE: now also D7.2 (A), R47.1, R48.1
- net HS_PULL: now also R48.2
- net LED_CLU: now also D10.2 (A), R52.2; no longer D8.2 (A)
- net LS_G: now also R49.2, R50.1
- net OA_FB: now also R54.2, R55.1, U9.4 (-)
- net OA_IN: now also C50.1, R53.2, U9.3 (+)
- net OA_OUT: now also R54.1, R56.1, U9.1; no longer R47.1
Other:
- moved on the sheet: D7, R47
Changed lines of the file:
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@@
 		(on_board yes)
 		(dnp no)
-		(property "Reference" "C32"
+		(property "Reference" "C49"
 			(at 58.42 66.675 0)
 			(effects
@@
 			(project "power-feed"
 				(path "/8e300617-3fca-5828-bedd-07eaa661f340/fee9f53f-ca95-5009-a118-475b15ee829d"
-					(reference "C32")
+					(reference "C49")
 					(unit 1)
 				)
@@
 		(on_board yes)
 		(dnp no)
-		(property "Reference" "R38"
+		(property "Reference" "R47"
 			(at 114.3 66.675 0)
 			(effects
@@
 			(project "power-feed"
 				(path "/8e300617-3fca-5828-bedd-07eaa661f340/fee9f53f-ca95-5009-a118-475b15ee829d"
-					(reference "R38")
+					(reference "R47")
 					(unit 1)
 				)
@@
 		(on_board yes)
 		(dnp no)
-		(property "Reference" "D5"
+		(property "Reference" "D7"
 			(at 147.32 66.675 0)
 			(effects
@@
 			(project "power-feed"
 				(path "/8e300617-3fca-5828-bedd-07eaa661f340/fee9f53f-ca95-5009-a118-475b15ee829d"
-					(reference "D5")
+					(reference "D7")
 					(unit 1)
 				)
@@
 		(on_board yes)
 		(dnp no)
-		(property "Reference" "R39"
+		(property "Reference" "R48"
 			(at 180.34 66.675 0)
 			(effects
@@
 			(project "power-feed"
 				(path "/8e300617-3fca-5828-bedd-07eaa661f340/fee9f53f-ca95-5009-a118-475b15ee829d"
-					(reference "R39")
+					(reference "R48")
 					(unit 1)
 				)
@@
 		(on_board yes)
 		(dnp no)
-		(property "Reference" "J3"
+		(property "Reference" "J5"
 			(at 38.1 96.52 0)
 			(effects
@@
 			(project "power-feed"
 				(path "/8e300617-3fca-5828-bedd-07eaa661f340/fee9f53f-ca95-5009-a118-475b15ee829d"
-					(reference "J3")
+					(reference "J5")
 					(unit 1)
 				)
@@
 		(on_board yes)
 		(dnp no)
-		(property "Reference" "D6"
+		(property "Reference" "D8"
 			(at 71.12 96.52 0)
 			(effects
@@
 			(project "power-feed"
 				(path "/8e300617-3fca-5828-bedd-07eaa661f340/fee9f53f-ca95-5009-a118-475b15ee829d"
-					(reference "D6")
+					(reference "D8")
 					(unit 1)
 				)
@@
 		(on_board yes)
 		(dnp no)
-		(property "Reference" "D7"
+		(property "Reference" "D9"
 			(at 109.22 96.52 0)
 			(effects
@@
 			(project "power-feed"
 				(path "/8e300617-3fca-5828-bedd-07eaa661f340/fee9f53f-ca95-5009-a118-475b15ee829d"
-					(reference "D7")
+					(reference "D9")
 					(unit 1)
 				)
@@
 		(on_board yes)
 		(dnp no)
-		(property "Reference" "R40"
+		(property "Reference" "R49"
 			(at 137.16 96.52 0)
 			(effects
@@
 			(project "power-feed"
 				(path "/8e300617-3fca-5828-bedd-07eaa661f340/fee9f53f-ca95-5009-a118-475b15ee829d"
-					(reference "R40")
+					(reference "R49")
 					(unit 1)
 				)
@@
 		(on_board yes)
 		(dnp no)
-		(property "Reference" "R41"
+		(property "Reference" "R50"
 			(at 160.02 96.52 0)
 			(effects
@@
 			(project "power-feed"
 				(path "/8e300617-3fca-5828-bedd-07eaa661f340/fee9f53f-ca95-5009-a118-475b15ee829d"
-					(reference "R41")
+					(reference "R50")
 					(unit 1)
 				)
@@
 		(on_board yes)
 		(dnp no)
-		(property "Reference" "R42"
+		(property "Reference" "R51"
 			(at 215.9 96.52 0)
 			(effects
@@
 			(project "power-feed"
 				(path "/8e300617-3fca-5828-bedd-07eaa661f340/fee9f53f-ca95-5009-a118-475b15ee829d"
-					(reference "R42")
+					(reference "R51")
 					(unit 1)
 				)
@@
 		(on_board yes)
 		(dnp no)
-		(property "Reference" "R43"
+		(property "Reference" "R52"
 			(at 238.76 96.52 0)
 			(effects
@@
 			(project "power-feed"
 				(path "/8e300617-3fca-5828-bedd-07eaa661f340/fee9f53f-ca95-5009-a118-475b15ee829d"
-					(reference "R43")
+					(reference "R52")
 					(unit 1)
 				)
@@
 		(on_board yes)
 		(dnp no)
-		(property "Reference" "D8"
+		(property "Reference" "D10"
 			(at 266.7 96.52 0)
 			(effects
@@
 			(project "power-feed"
 				(path "/8e300617-3fca-5828-bedd-07eaa661f340/fee9f53f-ca95-5009-a118-475b15ee829d"
-					(reference "D8")
+					(reference "D10")
 					(unit 1)
 				)
@@
 		(on_board yes)
 		(dnp no)
-		(property "Reference" "R44"
+		(property "Reference" "R53"
 			(at 31.115 129.54 0)
 			(effects
@@
 			(project "power-feed"
 				(path "/8e300617-3fca-5828-bedd-07eaa661f340/fee9f53f-ca95-5009-a118-475b15ee829d"
-					(reference "R44")
+					(reference "R53")
 					(unit 1)
 				)
@@
 		(on_board yes)
 		(dnp no)
-		(property "Reference" "C33"
+		(property "Reference" "C50"
 			(at 53.975 129.54 0)
 			(effects
@@
 			(project "power-feed"
 				(path "/8e300617-3fca-5828-bedd-07eaa661f340/fee9f53f-ca95-5009-a118-475b15ee829d"
-					(reference "C33")
+					(reference "C50")
 					(unit 1)
 				)
@@
 		(on_board yes)
 		(dnp no)
-		(property "Reference" "U6"
+		(property "Reference" "U9"
 			(at 84.455 129.54 0)
 			(effects
@@
 			(project "power-feed"
 				(path "/8e300617-3fca-5828-bedd-07eaa661f340/fee9f53f-ca95-5009-a118-475b15ee829d"
-					(reference "U6")
+					(reference "U9")
 					(unit 1)
 				)
@@
 		(on_board yes)
 		(dnp no)
-		(property "Reference" "C34"
+		(property "Reference" "C51"
 			(at 114.935 129.54 0)
 			(effects
@@
 			(project "power-feed"
 				(path "/8e300617-3fca-5828-bedd-07eaa661f340/fee9f53f-ca95-5009-a118-475b15ee829d"
-					(reference "C34")
+					(reference "C51")
 					(unit 1)
 				)
@@
 		(on_board yes)
 		(dnp no)
-		(property "Reference" "R45"
+		(property "Reference" "R54"
 			(at 137.795 129.54 0)
 			(effects
@@
 			(project "power-feed"
 				(path "/8e300617-3fca-5828-bedd-07eaa661f340/fee9f53f-ca95-5009-a118-475b15ee829d"
-					(reference "R45")
+					(reference "R54")
 					(unit 1)
 				)
@@
 		(on_board yes)
 		(dnp no)
-		(property "Reference" "R46"
+		(property "Reference" "R55"
 			(at 160.655 129.54 0)
 			(effects
@@
 			(project "power-feed"
 				(path "/8e300617-3fca-5828-bedd-07eaa661f340/fee9f53f-ca95-5009-a118-475b15ee829d"
-					(reference "R46")
+					(reference "R55")
 					(unit 1)
 				)
@@
 		(on_board yes)
 		(dnp no)
-		(property "Reference" "R47"
+		(property "Reference" "R56"
 			(at 183.515 129.54 0)
 			(effects
@@
 			(project "power-feed"
 				(path "/8e300617-3fca-5828-bedd-07eaa661f340/fee9f53f-ca95-5009-a118-475b15ee829d"
-					(reference "R47")
+					(reference "R56")
 					(unit 1)
 				)
@@
 		(on_board yes)
 		(dnp no)
-		(property "Reference" "C35"
+		(property "Reference" "C52"
 			(at 206.375 129.54 0)
 			(effects
@@
 			(project "power-feed"
 				(path "/8e300617-3fca-5828-bedd-07eaa661f340/fee9f53f-ca95-5009-a118-475b15ee829d"
-					(reference "C35")
+					(reference "C52")
 					(unit 1)
 				)

Commit message: Schematic: 100 nF right at RP2040 DVDD pin 23 and USBLC6-2SC6 ESD (C7519) on the USB-C lines (PCB review round 2)
Co-Authored-By: Claude Opus 5.5 <noreply@anthropic.com>
Parts:
- removed C49: 2.2uF 100V, Capacitor_SMD:C_1210_3225Metric, symbol Device:C
- removed U9: TLV9061, Package_TO_SOT_SMD:SOT-23-5, symbol Amplifier_Operational:TLV9061xDBV
- added C53: 10nF, Capacitor_SMD:C_0603_1608Metric, symbol Device:C
- added U10: TLV9061, Package_TO_SOT_SMD:SOT-23-5, symbol Amplifier_Operational:TLV9061xDBV
- C50: value 1nF -> 2.2uF 100V; footprint Capacitor_SMD:C_0603_1608Metric -> Capacitor_SMD:C_1210_3225Metric; LCSC C1588 -> C86054; MPN Samsung CL10B102KB8NNNC -> Murata GRM32ER72A225KA35L
- C51: value 100nF -> 1nF; LCSC C14663 -> C1588; MPN Yageo CC0603KRX7R9BB104 -> Samsung CL10B102KB8NNNC
- C52: value 10nF -> 100nF; LCSC C57112 -> C14663; MPN FH 0603B103K500NT -> Yageo CC0603KRX7R9BB104
Connections:
- net +3V3: now also C52.1, U10.5 (V+); no longer C51.1
- net CLUTCH_ISENSE: now also C53.1; no longer C52.1
- net CLUTCH_VIN: now also C50.1
- net GND: now also C53.2, U10.2 (V-)
- net OA_FB: now also U10.4 (-)
- net OA_IN: now also C51.1, U10.3 (+); no longer C50.1
- net OA_OUT: now also U10.1
Other:
- moved on the sheet: C50, C51, C52
Changed lines of the file:
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@@
 		(on_board yes)
 		(dnp no)
-		(property "Reference" "C49"
+		(property "Reference" "C50"
 			(at 58.42 66.675 0)
 			(effects
@@
 			(project "power-feed"
 				(path "/8e300617-3fca-5828-bedd-07eaa661f340/fee9f53f-ca95-5009-a118-475b15ee829d"
-					(reference "C49")
+					(reference "C50")
 					(unit 1)
 				)
@@
 		(on_board yes)
 		(dnp no)
-		(property "Reference" "C50"
+		(property "Reference" "C51"
 			(at 53.975 129.54 0)
 			(effects
@@
 			(project "power-feed"
 				(path "/8e300617-3fca-5828-bedd-07eaa661f340/fee9f53f-ca95-5009-a118-475b15ee829d"
-					(reference "C50")
+					(reference "C51")
 					(unit 1)
 				)
@@
 		(on_board yes)
 		(dnp no)
-		(property "Reference" "U9"
+		(property "Reference" "U10"
 			(at 84.455 129.54 0)
 			(effects
@@
 			(project "power-feed"
 				(path "/8e300617-3fca-5828-bedd-07eaa661f340/fee9f53f-ca95-5009-a118-475b15ee829d"
-					(reference "U9")
+					(reference "U10")
 					(unit 1)
 				)
@@
 		(on_board yes)
 		(dnp no)
-		(property "Reference" "C51"
+		(property "Reference" "C52"
 			(at 114.935 129.54 0)
 			(effects
@@
 			(project "power-feed"
 				(path "/8e300617-3fca-5828-bedd-07eaa661f340/fee9f53f-ca95-5009-a118-475b15ee829d"
-					(reference "C51")
+					(reference "C52")
 					(unit 1)
 				)
@@
 		(on_board yes)
 		(dnp no)
-		(property "Reference" "C52"
+		(property "Reference" "C53"
 			(at 206.375 129.54 0)
 			(effects
@@
 			(project "power-feed"
 				(path "/8e300617-3fca-5828-bedd-07eaa661f340/fee9f53f-ca95-5009-a118-475b15ee829d"
-					(reference "C52")
+					(reference "C53")
 					(unit 1)
 				)
